File: ESP32_Tasmota_Fan.sch (KiCad schematic (older format))
At the start: 12 parts, among them J1 Conn_01x02_Female, J3 Conn_01x10, Q1 AO3401A

Commit message: Version open for review
Connections:
- no-connect marks 0 -> 2
Other:
- moved on the sheet: D3, J1, Q1, R12
Changed lines of the file:
@@
 L Connector:Conn_01x02_Female J1
 U 1 1 605C2A51
-P 1050 1550
-F 0 "J1" H 942 1735 50  0000 C CNN
-F 1 "Conn_01x02_Female" H 942 1644 50  0000 C CNN
-F 2 "Connector_BarrelJack:BarrelJack_CUI_PJ-102AH_Horizontal" H 1050 1550 50  0001 C CNN
-F 3 "~" H 1050 1550 50  0001 C CNN
-	1    1050 1550
+P 950 1650
+F 0 "J1" H 842 1835 50  0000 C CNN
+F 1 "Conn_01x02_Female" H 842 1744 50  0000 C CNN
+F 2 "Connector_BarrelJack:BarrelJack_CUI_PJ-102AH_Horizontal" H 950 1650 50  0001 C CNN
+F 3 "~" H 950 1650 50  0001 C CNN
+	1    950  1650
 	-1   0    0    -1
 $EndComp
@@
 L power:GND #PWR07
 U 1 1 605C41B3
-P 1350 1700
-F 0 "#PWR07" H 1350 1450 50  0001 C CNN
-F 1 "GND" H 1355 1527 50  0000 C CNN
-F 2 "" H 1350 1700 50  0001 C CNN
-F 3 "" H 1350 1700 50  0001 C CNN
-	1    1350 1700
+P 1250 1900
+F 0 "#PWR07" H 1250 1650 50  0001 C CNN
+F 1 "GND" H 1255 1727 50  0000 C CNN
+F 2 "" H 1250 1900 50  0001 C CNN
+F 3 "" H 1250 1900 50  0001 C CNN
+	1    1250 1900
 	1    0    0    -1
 $EndComp
@@
 L power:+12V #PWR06
 U 1 1 605C4698
-P 2250 1450
-F 0 "#PWR06" H 2250 1300 50  0001 C CNN
-F 1 "+12V" H 2265 1623 50  0000 C CNN
-F 2 "" H 2250 1450 50  0001 C CNN
-F 3 "" H 2250 1450 50  0001 C CNN
-	1    2250 1450
-	1    0    0    -1
-$EndComp
-Wire Wire Line
-	1350 1650 1350 1700
+P 2150 1550
+F 0 "#PWR06" H 2150 1400 50  0001 C CNN
+F 1 "+12V" H 2165 1723 50  0000 C CNN
+F 2 "" H 2150 1550 50  0001 C CNN
+F 3 "" H 2150 1550 50  0001 C CNN
+	1    2150 1550
+	1    0    0    -1
+$EndComp
+Wire Wire Line
+	1250 1850 1250 1900
 $Comp
 L Mechanical:MountingHole H1
@@
 PSU Requirements\n3.3V @ 500mA
 Wire Wire Line
-	2250 1550 2250 1450
-Text Notes 950  1150 0    50   ~ 0
+	2150 1650 2150 1550
+Text Notes 850  1250 0    50   ~ 0
 Power Input\n12V 5.5mm/2.1mm Barrel Jack
 Text Notes 1050 5150 0    50   ~ 0
 Temperature Sensor Options - OneWire\nDHT22 - VCC/Data/NC/GND\nDS18B20 - VCC/Data/GND (leave one spare when connecting)
-Text Notes 3650 1100 0    50   ~ 0
+Text Notes 3550 1200 0    50   ~ 0
 LDO Option\n8,7V Voltagedrop\n500mA Iout\n4,35W Ploss
 $Sheet
-S 2950 1300 900  500
+S 2850 1400 900  500
 U 6192B19F
 F0 "DC/DC Buck" 50
 F1 "BuckConverter.sch" 50
-F2 "VOUT" I R 3850 1550 50
-F3 "VIN" I L 2950 1550 50
+F2 "VOUT" I R 3750 1650 50
+F3 "VIN" I L 2850 1650 50
 $EndSheet
 Wire Wire Line
-	3850 1550 4150 1550
-Wire Wire Line
-	4150 1550 4150 1450
+	3750 1650 4050 1650
+Wire Wire Line
+	4050 1650 4050 1550
 $Comp
 L power:+3V3 #PWR010
 U 1 1 618AE64B
-P 4150 1450
-F 0 "#PWR010" H 4150 1300 50  0001 C CNN
-F 1 "+3V3" H 4165 1623 50  0000 C CNN
-F 2 "" H 4150 1450 50  0001 C CNN
-F 3 "" H 4150 1450 50  0001 C CNN
-	1    4150 1450
+P 4050 1550
+F 0 "#PWR010" H 4050 1400 50  0001 C CNN
+F 1 "+3V3" H 4065 1723 50  0000 C CNN
+F 2 "" H 4050 1550 50  0001 C CNN
+F 3 "" H 4050 1550 50  0001 C CNN
+	1    4050 1550
 	1    0    0    -1
 $EndComp
@@
 L Device:D_Zener D3
 U 1 1 61921BA4
-P 2250 1750
-F 0 "D3" V 2204 1830 50  0000 L CNN
-F 1 "ZMM5V6" V 2295 1830 50  0000 L CNN
-F 2 "Diode_SMD:D_MiniMELF" H 2250 1750 50  0001 C CNN
-F 3 "~" H 2250 1750 50  0001 C CNN
-F 4 "C8062" V 2250 1750 50  0001 C CNN "LCSC"
-	1    2250 1750
+P 2150 1850
+F 0 "D3" V 2104 1930 50  0000 L CNN
+F 1 "ZMM5V6" V 2195 1930 50  0000 L CNN
+F 2 "Diode_SMD:D_MiniMELF" H 2150 1850 50  0001 C CNN
+F 3 "~" H 2150 1850 50  0001 C CNN
+F 4 "C8062" V 2150 1850 50  0001 C CNN "LCSC"
+	1    2150 1850
 	0    1    1    0
 $EndComp
@@
 L Device:R_Small R12
 U 1 1 619229FB
-P 1900 2100
-F 0 "R12" H 1959 2146 50  0000 L CNN
-F 1 "100R" H 1959 2055 50  0000 L CNN
-F 2 "Resistor_SMD:R_0805_2012Metric" H 1900 2100 50  0001 C CNN
-F 3 "~" H 1900 2100 50  0001 C CNN
-F 4 "C17408" H 1900 2100 50  0001 C CNN "LCSC"
-	1    1900 2100
+P 1800 2200
+F 0 "R12" H 1859 2246 50  0000 L CNN
+F 1 "100R" H 1859 2155 50  0000 L CNN
+F 2 "Resistor_SMD:R_0805_2012Metric" H 1800 2200 50  0001 C CNN
+F 3 "~" H 1800 2200 50  0001 C CNN
+F 4 "C17408" H 1800 2200 50  0001 C CNN "LCSC"
+	1    1800 2200
 	1    0    0    -1
 $EndComp
@@
 L power:GND #PWR01
 U 1 1 61924CDE
-P 1900 2250
-F 0 "#PWR01" H 1900 2000 50  0001 C CNN
-F 1 "GND" H 1905 2077 50  0000 C CNN
-F 2 "" H 1900 2250 50  0001 C CNN
-F 3 "" H 1900 2250 50  0001 C CNN
-	1    1900 2250
-	1    0    0    -1
-$EndComp
-Wire Wire Line
-	1250 1650 1350 1650
-Wire Wire Line
-	1900 2250 1900 2200
-Wire Wire Line
-	1900 2000 1900 1950
-Wire Wire Line
-	1900 1950 2250 1950
-Wire Wire Line
-	2250 1950 2250 1900
+P 1800 2350
+F 0 "#PWR01" H 1800 2100 50  0001 C CNN
+F 1 "GND" H 1805 2177 50  0000 C CNN
+F 2 "" H 1800 2350 50  0001 C CNN
+F 3 "" H 1800 2350 50  0001 C CNN
+	1    1800 2350
+	1    0    0    -1
+$EndComp
+Wire Wire Line
+	1800 2350 1800 2300
+Wire Wire Line
+	1800 2100 1800 2050
+Wire Wire Line
+	1800 2050 2150 2050
+Wire Wire Line
+	2150 2050 2150 2000
 $Comp
 L Transistor_FET:AO3401A Q1
 U 1 1 6192EDCC
-P 1900 1650
-F 0 "Q1" V 2242 1650 50  0000 C CNN
-F 1 "AO3401A" V 2151 1650 50  0000 C CNN
-F 2 "Package_TO_SOT_SMD:SOT-23" H 2100 1575 50  0001 L CIN
-F 3 "http://www.aosmd.com/pdfs/datasheet/AO3401A.pdf" H 1900 1650 50  0001 L CNN
-F 4 "C15127" V 1900 1650 50  0001 C CNN "LCSC"
-	1    1900 1650
+P 1800 1750
+F 0 "Q1" V 2142 1750 50  0000 C CNN
+F 1 "AO3401A" V 2051 1750 50  0000 C CNN
+F 2 "Package_TO_SOT_SMD:SOT-23" H 2000 1675 50  0001 L CIN
+F 3 "http://www.aosmd.com/pdfs/datasheet/AO3401A.pdf" H 1800 1750 50  0001 L CNN
+F 4 "C15127" V 1800 1750 50  0001 C CNN "LCSC"
+	1    1800 1750
 	0    -1   -1   0
 $EndComp
 Wire Wire Line
-	2100 1550 2250 1550
-Wire Wire Line
-	2250 1550 2250 1600
-Wire Wire Line
-	1900 1850 1900 1950
-Connection ~ 1900 1950
-Wire Wire Line
-	1250 1550 1700 1550
-Connection ~ 2250 1550
-Wire Wire Line
-	2250 1550 2950 1550
-Text Label 1250 1550 0    50   ~ 0
+	2000 1650 2150 1650
+Wire Wire Line
+	2150 1650 2150 1700
+Wire Wire Line
+	1800 1950 1800 2050
+Connection ~ 1800 2050
+Connection ~ 2150 1650
+Wire Wire Line
+	2150 1650 2500 1650
+Text Label 1150 1650 0    50   ~ 0
 VIN
 Wire Wire Line
@@
 Text Notes 9400 750  2    118  ~ 24
 FANS
+Wire Wire Line
+	6300 1700 6400 1700
+Wire Wire Line
+	7700 1400 7600 1400
+NoConn ~ 7700 1400
+NoConn ~ 6300 1700
+$Comp
+L power:PWR_FLAG #FLG0103
+U 1 1 6192E948
+P 2500 1650
+F 0 "#FLG0103" H 2500 1725 50  0001 C CNN
+F 1 "PWR_FLAG" H 2500 1823 50  0000 C CNN
+F 2 "" H 2500 1650 50  0001 C CNN
+F 3 "~" H 2500 1650 50  0001 C CNN
+	1    2500 1650
+	1    0    0    -1
+$EndComp
+$Comp
+L power:PWR_FLAG #FLG0104
+U 1 1 6192FEED
+P 4050 1650
+F 0 "#FLG0104" H 4050 1725 50  0001 C CNN
+F 1 "PWR_FLAG" H 4050 1823 50  0000 C CNN
+F 2 "" H 4050 1650 50  0001 C CNN
+F 3 "~" H 4050 1650 50  0001 C CNN
+	1    4050 1650
+	0    1    1    0
+$EndComp
+Connection ~ 2500 1650
+Wire Wire Line
+	2500 1650 2850 1650
+Connection ~ 4050 1650
+Wire Wire Line
+	1150 1650 1600 1650
+$Comp
+L power:PWR_FLAG #FLG0101
+U 1 1 61934EDD
+P 1250 1850
+F 0 "#FLG0101" H 1250 1925 50  0001 C CNN
+F 1 "PWR_FLAG" H 1250 2023 50  0000 C CNN
+F 2 "" H 1250 1850 50  0001 C CNN
+F 3 "~" H 1250 1850 50  0001 C CNN
+	1    1250 1850
+	0    1    1    0
+$EndComp
+Wire Wire Line
+	1150 1750 1250 1750
+Wire Wire Line
+	1250 1750 1250 1850
+Connection ~ 1250 1850
 $EndSCHEMATC
